File: UINIO-Logic-24MHz.kicad_sch (KiCad schematic)
At the start: 51 parts, among them J1 Conn_01x10_Pin, U1 AT24CS64-XHM, U2 74HC245C, U3 ME6211C33M5G-N, U4 CY7C68013A-56LTX, Y1 24MHz

Commit message: chore: update parts
Parts:
- C1, C2: LCSC Part # (none) -> C15849
- C10: LCSC Part # (none) -> C52923
- C11, C12, C3, C4, C5, C6, C7: LCSC Part # (none) -> C1525
- C8, C9: LCSC Part # (none) -> C1547
- D1: LCSC Part # (none) -> C2286
- D2: LCSC Part # (none) -> C89811
- D3: LCSC Part # (none) -> C19189745
- D4: value 1N4007 -> 1N4007W; LCSC Part # (none) -> C18199088
- D5, D6: LCSC Part # (none) -> C5199850
- F1: LCSC Part # (none) -> C151135
- R1, R2, R3, R4, R5, R6, R7, R8: LCSC Part # (none) -> C25076
- R10, R11, R12, R13, R14, R15, R16, R23, R9: LCSC Part # (none) -> C25741
- R17: LCSC Part # (none) -> C11702
- R18, R19, R20: LCSC Part # (none) -> C25744
- R21, R22: LCSC Part # (none) -> C25879
- R24, R25: LCSC Part # (none) -> C23186
- U1: value AT24CS64-XHM -> AT24C64D-XHM-T; LCSC Part # (none) -> C111440
- U2: value 74HC245C -> 74HC245PW,118; symbol Uinio:74HC245C -> Uinio:74HC245; LCSC Part # (none) -> C5626; SuppliersPartNumber C126198 -> (none)
- U3: BOM名称 低功耗LDO -> (none); LCSC Part # (none) -> C82942
- U4: value CY7C68013A-56LTX -> CY7C68013A-56LTXC; LCSC Part # (none) -> C14912
- USB1: LCSC Part # (none) -> C2835315; SuppliersPartNumber C2835315 -> (none)
- Y1: LCSC Part # (none) -> C362340
Other:
- note added: "CY7C68013A USB2.0"
- note added: "EEPROM"
- note added: "LDO"
- note added: "USB Type-C"
- note added: "pull-up resistor"
- note added: "signal transceiver"
- note removed: "CY7C68013A USB2.0 控制器"
- note removed: "EEPROM 存储器"
- note removed: "LDO 线性稳压电路"
- note removed: "USB Type-C 接口电路"
- note removed: "上拉电阻"
- note removed: "信 号 收 发 器"

Commit message: fix: production check
Parts:
- removed D2: LED Yellow, LED_SMD:LED_0603_1608Metric, symbol Device:LED
- removed D3: LED Green, LED_SMD:LED_0603_1608Metric, symbol Device:LED
- removed D4: 1N4007W, Diode_SMD:Nexperia_CFP3_SOD-123W, symbol Diode:1N4007
- removed D5, D6: LESD5D5.0CT1G, Diode_SMD:D_SOD-523, symbol Diode:1N630xCA
- removed F1: 60V 1A, Fuse:Fuse_1206_3216Metric, symbol Device:Fuse
- removed R18, R19: 10K, Resistor_SMD:R_0402_1005Metric, symbol Device:R
- added C13, C14, C15: 0.1uF, Capacitor_SMD:C_0402_1005Metric, symbol Device:C
- added C16: 10uF, Capacitor_SMD:C_0805_2012Metric, symbol Device:C
- added J2: Conn_01x03, Connector_PinHeader_2.54mm:PinHeader_1x03_P2.54mm_Vertical, symbol Connector_Generic:Conn_01x03
- added J3: GPIO, Connector_PinHeader_2.54mm:PinHeader_1x10_P2.54mm_Vertical, symbol Connector:Conn_01x10_Pin
- U2: value 74HC245PW,118 -> 74LVC245APW,118; LCSC Part # C5626 -> C6082
- Y1: footprint Crystal:Crystal_SMD_3225-4Pin_3.2x2.5mm -> Uinio:HC-49-SMD_L7.0-W3.0; symbol Device:Crystal_GND24 -> Uinio:X49XM24MOB2SC; LCSC Part # C362340 -> C412889; MPN (none) -> X49XM24MOB2SC; Manufacturer (none) -> YXC
Connections:
- net +3.3V: now also C2.2, U3.5 (Vout), C13.2, C14.2, C15.1, C16.1, J2.3 (Pin_3), J3.10 (Pin_10)
- net GND: now also C13.1, C14.1, C15.2, C16.2, J2.1 (Pin_1), J3.9 (Pin_9); no longer U1.1 (A0), Y1.2, Y1.4
- net at C8.2, U4.4 (XTALOUT): now also Y1.2 (OSC2); no longer Y1.3
- net PA0: now reaches U4.33 (PA0/~{INT0})
- net PA0: now also J3.1 (Pin_1)
- net PA1: now reaches U4.34 (PA1/~{INT1})
- net PA1: now also J3.2 (Pin_2)
- net PA2: now reaches U4.35 (PA2/SLOE)
- net PA2: now also J3.3 (Pin_3)
- net PA3: now reaches U4.36 (PA3/WU2)
- net PA3: now also J3.4 (Pin_4)
- net PA4: now reaches U4.37 (PA4/FIOADDR0)
- net PA4: now also J3.5 (Pin_5)
- net PA5: now reaches U4.38 (PA5/FIOADDR1)
- net PA5: now also J3.6 (Pin_6)
- net PA6: now reaches U4.39 (PA6/PKTEND)
- net PA6: now also J3.7 (Pin_7)
- net PA7: now reaches U4.40 (PA7/FLAGD/~{SLCS})
- net PA7: now also J3.8 (Pin_8)
- new net: J2.2 (Pin_2), U1.1 (A0)
- no-connect marks 24 -> 18
Other:
- moved on the sheet: C11, C12, C3, C4, C5, C6, C7, J1
