File: UINIO-Logic-24MHz.kicad_pcb (KiCad board)
At the start: 2 copper layers, 52 x 25.4 mm, 55 parts, among them J1 Conn_01x10_Pin, U1 AT24CS64-XHM, U2 74HC245C, U3 ME6211C33M5G-N, U4 CY7C68013A-56LTX, Y1 24MHz

Commit message: chore: update parts
Parts:
- D4: value 1N4007 -> 1N4007W
- U1: value AT24CS64-XHM -> AT24C64D-XHM-T
- U2: value 74HC245C -> 74HC245PW,118
- U4: value CY7C68013A-56LTX -> CY7C68013A-56LTXC

Commit message: feat: update silkscreen
Parts:
- added G***: LOGO, LOGO, B.Cu at (149.2, 106.3)
Other:
- board text removed: "UINIO Logic 24MHz"
- board text removed: "UINIO-Logic-24MHz"
- board text removed: "UinIO.com"
- board text removed: "Version 5.0.0"

Commit message: fix: production check
Parts:
- removed D2: LED Yellow, LED_SMD:LED_0603_1608Metric
- removed D3: LED Green, LED_SMD:LED_0603_1608Metric
- removed D4: 1N4007W, Diode_SMD:Nexperia_CFP3_SOD-123W
- removed D5, D6: LESD5D5.0CT1G, Diode_SMD:D_SOD-523
- removed F1: 60V 1A, Fuse:Fuse_1206_3216Metric
- removed R18, R19: 10K, Resistor_SMD:R_0402_1005Metric
- added C13: 0.1uF, Capacitor_SMD:C_0402_1005Metric, F.Cu at (158.4, 101.5)
- added C14: 0.1uF, Capacitor_SMD:C_0402_1005Metric, F.Cu at (155.3, 111.9)
- added C15: 0.1uF, Capacitor_SMD:C_0402_1005Metric, F.Cu at (140.1, 101.7)
- added C16: 10uF, Capacitor_SMD:C_0805_2012Metric, F.Cu at (152.3, 101.8)
- added J2: Conn_01x03, Connector_PinHeader_2.54mm:PinHeader_1x03_P2.54mm_Vertical, F.Cu at (162.2, 115.0)
- added J3: GPIO, Connector_PinHeader_2.54mm:PinHeader_1x10_P2.54mm_Vertical, F.Cu at (156.8, 96.2)
- U2: value 74HC245PW,118 -> 74LVC245APW,118
- Y1: footprint Crystal:Crystal_SMD_3225-4Pin_3.2x2.5mm -> Uinio:HC-49-SMD_L7.0-W3.0
- moved R16 18.3 mm to (156.7, 99.0), turned to -90 degrees
- moved R15 17.5 mm to (157.7, 99.0), turned to -90 degrees
- moved R14 17.0 mm to (158.7, 99.0), turned to -90 degrees
- moved R13 16.9 mm to (159.7, 99.0), turned to -90 degrees
- moved R17 16.2 mm to (135.6, 100.1), turned to 90 degrees
- moved D1 14.0 mm to (133.6, 100.3), turned to 0 degrees
- moved C9 12.0 mm to (136.6, 111.1), turned to 90 degrees
- moved C1 9.69 mm to (147.0, 115.3)
- moved C2 9.69 mm to (152.7, 115.3)
- moved U3 9.69 mm to (149.8, 115.0)
- moved Y1 9.17 mm to (136.6, 105.6), turned to 90 degrees
- moved R25 5.66 mm to (129.3, 111.6)
- moved R24 5.63 mm to (129.3, 99.6)
- moved R23 5.29 mm to (138.5, 100.1), turned to -90 degrees
- moved C10 4.71 mm to (137.6, 100.1), turned to 90 degrees
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Connections:
- C2 pad 2: Net-(U3-Vout) -> +3.3V
- U1 pad 1: GND -> Net-(J2-Pin_2)
- U3 pad 5: Net-(U3-Vout) -> +3.3V
- U4 pad 33: Net-(U4-PA0/~{INT0}) -> /PA0
- U4 pad 34: Net-(U4-PA1/~{INT1}) -> /PA1
- U4 pad 35: unconnected-(U4-PA2/SLOE-Pad35) -> /PA2
- U4 pad 36: unconnected-(U4-PA3/WU2-Pad36) -> /PA3
- U4 pad 37: unconnected-(U4-PA4/FIOADDR0-Pad37) -> /PA4
- U4 pad 38: unconnected-(U4-PA5/FIOADDR1-Pad38) -> /PA5
- U4 pad 39: unconnected-(U4-PA6/PKTEND-Pad39) -> /PA6
- U4 pad 40: unconnected-(U4-PA7/FLAGD/~{SLCS}-Pad40) -> /PA7
- Y1 pad 2: GND -> Net-(U4-XTALOUT)
Routing:
- net +3.3V: track 167.8 -> 110.2 mm, vias 12 -> 18
- net +5V: track 2.52 -> 35.9 mm, vias 5 -> 6
- net /PA0: track 0.00 -> 14.0 mm
- net Net-(U4-PA0/~{INT0}): track 12.2 -> 0.00 mm
- net /PA1: track 0.00 -> 11.9 mm
- net /PA2: track 0.00 -> 9.96 mm
- net Net-(U4-XTALIN): track 24.0 -> 15.1 mm
- net /PA3: track 0.00 -> 8.50 mm
- net /PA7: track 0.00 -> 7.65 mm
- net Net-(U4-PA1/~{INT1}): track 6.31 -> 0.00 mm
- net /PA4: track 0.00 -> 6.31 mm
- net /PA6: track 0.00 -> 6.30 mm
- net Net-(J2-Pin_2): track 0.00 -> 5.65 mm
- net /PA5: track 0.00 -> 5.47 mm
- net /INPUT8: track 12.5 -> 17.3 mm
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- removed copper zone on F.Cu, net Net-(U3-Vout)
Other:
- board text added: "0"
- board text added: "1"
- board text added: "2026"
- board text added: "woldhack"
- board text removed: "PA0"
- board text removed: "PA1"
- board text removed: "Power"

Commit message: feat: update silkscreen
Parts:
- moved C13 2.28 mm to (160.6, 101.6), turned to 0 degrees
- moved G*** 0.90 mm to (149.3, 107.2)
Routing:
- net +3.3V: track 110.2 -> 111.1 mm
- net GND: vias 76 -> 86
